File: hardware/SATVIK-26/SATVIK-26.kicad_sch (KiCad schematic)
At the start: 6 parts, among them U1 SST26VF064Bxx-xxxx-MF

Commit message: CubeMX
Parts:
- added R3, R4, R5, R6, R7, R8, R9: R, symbol Device:R
Connections:
- net at C1.1: now also C2.1
- net at C1.2: now also R2.1
- net at R2.2: now also R3.1
- net at C2.2: now also R3.2
- new net: R7.2, R9.2
- new net: R8.2, R9.1
Other:
- moved on the sheet: C3, R1, U1
