File: hardware/SATVIK-26/SATVIK-26.kicad_sch (KiCad schematic)
At the start: 23 parts, among them SW1 SW_Push, SW2 SW_Push, U1 STM32H743VITx, U2 TPS54560BDDA, Y1 Crystal

Commit message: Cezual update
Parts:
- added C16: 100nF, symbol Device:C
- added C17, C18: 47uF, symbol Device:C
- added C19: 3.3nF, symbol Device:C
- added C20: 100pF, symbol Device:C
- added C21, C22: 1uF, symbol Device:C
- added D1: B560/SS56, symbol Device:D_Schottky
- added D2: SMBJ26A, symbol Device:D_TVS
- added L1: 15uH, symbol Device:L
- added R4: 100k, symbol Device:R
- added R5: 52.3k, symbol Device:R
- added R6: 10k, symbol Device:R
- added R7: 4.99k, symbol Device:R
- added R8: R, symbol Device:R
- added U3: AP2112K-3.3, Package_TO_SOT_SMD:SOT-23-5, symbol Regulator_Linear:AP2112K-3.3
Connections:
- net +3V3: now also U1.100 (VDD), U1.11 (VDD), U1.21 (VDDA), U1.27 (VDD), U1.50 (VDD), U1.6 (VBAT), U1.75 (VDD), C22.1, U3.5 (VOUT)
- net GND: now also U2.7 (GND), U2.9 (GND), C17.2, C18.2, C19.2, C20.2, C21.1, C22.2, D1.2 (A), D2.2 (A2), R4.2, R6.1, U3.2 (GND)
- net at C6.2, C7.2, C9.2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: now also D2.1 (A1)
- net at U2.1 (BOOT): now also C16.1
- net at U2.4 (RT/CLK): now also R4.1
- net at U2.5 (FB): now also R5.2, R6.2
- net at U2.6 (COMP): now also C20.1, R7.1
- net at U2.8 (SW): now also C16.2, D1.1 (K), L1.1
- net at U1.15 (PC0): now also R8.2
- new net: C19.1, R7.2
- new net +5V: C17.1, C18.1, C21.2, L1.2, R5.1, U3.1 (VIN), U3.3 (EN)
Other:
- moved on the sheet: C10, C11, C12, C13, C14, C15, C6, C7, C8, C9, R2, R3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

Commit message: couple hours
Parts:
- added C23, C24, C25, C26, C27, C28, C29: 100nF, symbol Device:C
- added J1: Micro_SD_Card_Det1, Connector_Card:microSD_HC_Hirose_DM3AT-SF-PEJM5, symbol Connector:Micro_SD_Card_Det1
- added R10, R11: 4.7k, symbol Device:R
- added R12, R13: 5.1k, symbol Device:R
- added R14, R15, R16, R17, R18: 47k, symbol Device:R
- added R9: 1k, symbol Device:R
- added U4: ICM-42688-P, easyeda2kicad:LGA-14_L3.0-W2.5-P0.50-TL, symbol easyeda2kicad:ICM-42688-P
- added U5: BMP388, easyeda2kicad:SENSORM-SMD_BMP388, symbol easyeda2kicad:BMP388
- added U6: USBLC6-2SC6, Package_TO_SOT_SMD:SOT-23-6, symbol Power_Protection:USBLC6-2SC6
- added USB1: TYPE-C 16PIN 2MD, easyeda2kicad:USB-C-SMD_TYPE-C-16PIN-2MD-073, symbol easyeda2kicad:TYPE-C16PIN2MD
- R8: value R -> 10k
Connections:
- net +3V3: now also C25.1, C26.1, C27.1, C28.2, C29.1, J1.4 (VDD), R10.2, R11.2, R14.2, R15.2, R16.2, R17.2, R18.2, U4.5 (VDDIO), U4.8 (VDD), U5.1 (VDDIO), U5.10 (VDD), U5.6 (CSB)
- net GND: now also C23.2, C24.1, C25.2, C26.2, C27.2, C28.1, C29.2, J1.6 (VSS), J1.SH (SHIELD), R12.2, R13.2, R9.2, U4.6 (GND), U5.3 (VSS), U5.5 (SDO), U5.8 (VSS), U5.9 (VSS), U6.2 (GND), USB1.13 (EH), USB1.14 (EH), USB1.A1B12 (GND), USB1.B1A12 (GND)
- net VBAT_RAW: now reaches C6.2, C7.2, C9.2, D2.1 (A1), R2.1, U2.2 (VIN)
- net VBAT_RAW: now also R8.2
- net at R8.1: now also U1.15 (PC0), C23.1, R9.1
- net CURR: now reaches U1.16 (PC1)
- net CURR: now also C24.2
- net SPI1_SCLK: now reaches U1.29 (PA5)
- net SPI1_SCLK: now also U4.13 (AP_SCL/AP_SCLK)
- net SPI1_MISO: now reaches U1.30 (PA6)
- net SPI1_MISO: now also U4.1 (AP_SDO/AP_AD0)
- net SPI1_MOSI: now reaches U1.31 (PA7)
- net SPI1_MOSI: now also U4.14 (AP_SDA/AP_SDIO/AP_SDI)
- net I2C2_SCL: now reaches U1.46 (PB10)
- net I2C2_SCL: now also R10.1, U5.2 (SCK)
- net I2C2_SDA: now reaches U1.47 (PB11)
- net I2C2_SDA: now also R11.1, U5.4 (SDI)
- net SD_D0: now reaches U1.65 (PC8)
- net SD_D0: now also J1.7 (DAT0), R14.1
- net SD_D1: now reaches U1.66 (PC9)
- net SD_D1: now also J1.8 (DAT1), R18.1
- net SD_DET: now reaches U1.7 (PC13)
- net SD_DET: now also J1.9 (DET)
- net USB_DM_MCU: now reaches U1.70 (PA11)
- net USB_DM_MCU: now also U6.4 (I/O2)
- net USB_DP_MCU: now reaches U1.71 (PA12)
- net USB_DP_MCU: now also U6.6 (I/O1)
- net SD_D2: now reaches U1.78 (PC10)
- net SD_D2: now also J1.1 (DAT2), R17.1
- net SD_D3: now reaches U1.79 (PC11)
- net SD_D3: now also J1.2 (DAT3/CD), R16.1
- net SD_CLK: now reaches U1.80 (PC12)
- net SD_CLK: now also J1.5 (CLK)
- net SD_CMD: now reaches U1.83 (PD2)
- net SD_CMD: now also J1.3 (CMD), R15.1
- net IMU_CS: now reaches U1.9 (PC15)
- net IMU_CS: now also U4.12 (AP_CS)
- new net: R13.1, USB1.A5 (CC1)
- new net: R12.1, USB1.B5 (CC2)
- new net USB_DM: U6.3 (I/O2), USB1.A7 (Dn1), USB1.B7 (Dn2)
- new net USB_DP: U6.1 (I/O1), USB1.A6 (Dp1), USB1.B6 (Dp2)
- new net VBUS: U6.5 (VBUS), USB1.A4B9 (VBUS), USB1.B4A9 (VBUS)
Other:
- moved on the sheet: R8

Commit message: Schematic Completed finally
Parts:
- added C30: 1uF, symbol Device:C
- added D3, D4, D5: LED, symbol Device:LED
- added J2: Conn_01x08_Pin, symbol Connector:Conn_01x08_Pin
- added J3: Conn_01x06_Pin, symbol Connector:Conn_01x06_Pin
- added J4: Conn_01x03_Pin, symbol Connector:Conn_01x03_Pin
- added J5, J6, J7: Conn_01x04_Pin, symbol Connector:Conn_01x04_Pin
- added R19: 47k, symbol Device:R
- added R20, R21: 1k, symbol Device:R
- added R22, R23: 330, symbol Device:R
Connections:
- net +3V3: now also R19.2, R21.2
- net +5V: now also C30.1, J3.1 (Pin_1), J4.1 (Pin_1), J5.1 (Pin_1), J6.1 (Pin_1), J7.1 (Pin_1), R20.2
- net CURR: now also J2.2 (Pin_2)
- net GND: now also C30.2, D3.1 (K), D4.1 (K), D5.1 (K), J2.8 (Pin_8), J3.2 (Pin_2), J4.3 (Pin_3), J5.2 (Pin_2), J6.2 (Pin_2), J7.2 (Pin_2)
- net I2C2_SCL: now also J3.5 (Pin_5)
- net I2C2_SDA: now also J3.6 (Pin_6)
- net SD_DET: now also R19.1
- net VBAT_RAW: now also J2.1 (Pin_1)
- net MOTOR1: now reaches U1.22 (PA0)
- net MOTOR1: now also J2.4 (Pin_4)
- net MOTOR2: now reaches U1.23 (PA1)
- net MOTOR2: now also J2.5 (Pin_5)
- net MOTOR3: now reaches U1.24 (PA2)
- net MOTOR3: now also J2.6 (Pin_6)
- net MOTOR4: now reaches U1.25 (PA3)
- net MOTOR4: now also J2.7 (Pin_7)
- net at U1.34 (PB0): now also R23.1
- net LED_STATUS: now reaches U1.35 (PB1)
- net LED_STATUS: now also R22.2
- net USART7_RX: now reaches U1.37 (PE7)
- net USART7_RX: now also J7.4 (Pin_4)
- net USART7_TX: now reaches U1.38 (PE8)
- net USART7_TX: now also J7.3 (Pin_3)
- net USART6_TX: now reaches U1.63 (PC6)
- net USART6_TX: now also J5.3 (Pin_3)
- net USART6_RX: now reaches U1.64 (PC7)
- net USART6_RX: now also J5.4 (Pin_4)
- net USART1_TX: now reaches U1.68 (PA9)
- net USART1_TX: now also J6.3 (Pin_3)
- net USART1_RX: now reaches U1.69 (PA10)
- net USART1_RX: now also J6.4 (Pin_4)
- net USART2_TX: now reaches U1.86 (PD5)
- net USART2_TX: now also J3.3 (Pin_3)
- net USART2_RX: now reaches U1.87 (PD6)
- net USART2_RX: now also J3.4 (Pin_4)
- net UART4_RX: now reaches U1.95 (PB8)
- net UART4_RX: now also J2.3 (Pin_3)
- new net: D5.2 (A), R22.1
- new net: D3.2 (A), R20.1
- new net: D4.2 (A), R21.1
- new net WS2812_DATA: J4.2 (Pin_2), R23.2
- no-connect marks 0 -> 58
Other:
- moved on the sheet: C1, C10, C11, C12, C13, C14, C15, C16, C17, C18, C19, C2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

Commit message: bruh
tis shi is hard :)
Parts:
- C1, C10, C11, C12, C13, C16, C19, C2, C20, C21, C22, C23, C24, C25, C26, C27, C28, C29, C3, C30, C8, C9: footprint (none) -> Capacitor_SMD:C_0402_1005Metric
- C14, C15: footprint (none) -> Capacitor_SMD:C_0603_1608Metric
- C17, C18, C6, C7: footprint (none) -> Capacitor_SMD:C_1206_3216Metric
- C4, C5: value 20pF -> 15pF; footprint (none) -> Capacitor_SMD:C_0402_1005Metric
- D1: footprint (none) -> Diode_SMD:D_SMA
- D2: footprint (none) -> Diode_SMD:D_SMB
- D3, D4, D5: footprint (none) -> LED_SMD:LED_0603_1608Metric
- J2: footprint (none) -> Connector_JST:JST_GH_SM08B-GHS-TB_1x08-1MP_P1.25mm_Horizontal
- J3: footprint (none) -> Connector_JST:JST_GH_SM06B-GHS-TB_1x06-1MP_P1.25mm_Horizontal
- J4: footprint (none) -> Connector_JST:JST_GH_SM03B-GHS-TB_1x03-1MP_P1.25mm_Horizontal
- J5, J6, J7: footprint (none) -> Connector_JST:JST_GH_SM04B-GHS-TB_1x04-1MP_P1.25mm_Horizontal
- L1: footprint (none) -> easyeda2kicad:IND-SMD_L10.4-W10.3
- R1, R10, R11, R12, R13, R14, R15, R16, R17, R18, R19, R2, R20, R21, R22, R23, R3, R4, R5, R6, R7, R8, R9: footprint (none) -> Resistor_SMD:R_0402_1005Metric
- SW1, SW2: footprint (none) -> easyeda2kicad:SW-SMD_4P-L5.1-W5.1-P3.70-LS6.5-TL_H1.5
- Y1: footprint (none) -> easyeda2kicad:CRYSTAL-SMD_4P-L3.2-W2.5-BL

Commit message: finnaly
Connections:
- net GND: now also U4.10 (RESV), U4.11 (RESV), U4.2 (RESV), U4.3 (RESV), U4.7 (RESV), U4.9 (INT2/FSYNC/CLKIN)
- no-connect marks 58 -> 52
