File: hardware/SATVIK-26/_autosave-SATVIK-26.kicad_sch (KiCad schematic)
At the start: 23 parts, among them SW1 SW_Push, SW2 SW_Push, U1 STM32H743VITx, U2 TPS54560BDDA, Y1 Crystal

Commit message: backup
Connections:
- net +3V3: now also U1.100 (VDD), U1.11 (VDD), U1.21 (VDDA), U1.27 (VDD), U1.50 (VDD), U1.6 (VBAT), U1.75 (VDD)
Changed lines of the file:
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@@
+	)
+	(junction
+		(at 287.02 109.22)
+		(diameter 0)
+		(color 0 0 0 0)
 	)
 	(junction
@@
 	)
 	(junction
+		(at 294.64 109.22)
+		(diameter 0)
+		(color 0 0 0 0)
+	)
+	(junction
 		(at 266.7 128.27)
 		(diameter 0)
@@
 	)
 	(junction
+		(at 284.48 109.22)
+		(diameter 0)
+		(color 0 0 0 0)
+	)
+	(junction
 		(at 290.83 95.25)
 		(diameter 0)
@@
 		(color 0 0 0 0)
 	)
+	(junction
+		(at 289.56 109.22)
+		(diameter 0)
+		(color 0 0 0 0)
+	)
+	(junction
+		(at 292.1 109.22)
+		(diameter 0)
+		(color 0 0 0 0)
+	)
 	(wire
 		(pts
@@
 	(wire
 		(pts
+			(xy 281.94 113.03) (xy 281.94 109.22)
+		)
+		(stroke
+			(width 0)
+			(type default)
+		)
+	)
+	(wire
+		(pts
 			(xy 281.94 95.25) (xy 290.83 95.25)
 		)
@@
 	(wire
 		(pts
+			(xy 294.64 109.22) (xy 297.18 109.22)
+		)
+		(stroke
+			(width 0)
+			(type default)
+		)
+	)
+	(wire
+		(pts
 			(xy 149.86 190.5) (xy 149.86 189.23)
 		)
@@
 	(wire
 		(pts
+			(xy 292.1 109.22) (xy 294.64 109.22)
+		)
+		(stroke
+			(width 0)
+			(type default)
+		)
+	)
+	(wire
+		(pts
 			(xy 149.86 190.5) (xy 156.21 190.5)
 		)
@@
 	(wire
 		(pts
+			(xy 289.56 105.41) (xy 289.56 109.22)
+		)
+		(stroke
+			(width 0)
+			(type default)
+		)
+	)
+	(wire
+		(pts
+			(xy 297.18 109.22) (xy 297.18 113.03)
+		)
+		(stroke
+			(width 0)
+			(type default)
+		)
+	)
+	(wire
+		(pts
 			(xy 142.24 207.01) (xy 142.24 212.09)
 		)
@@
 	(wire
 		(pts
+			(xy 289.56 109.22) (xy 292.1 109.22)
+		)
+		(stroke
+			(width 0)
+			(type default)
+		)
+	)
+	(wire
+		(pts
 			(xy 245.11 153.67) (xy 248.92 153.67)
 		)
@@
 	(wire
 		(pts
+			(xy 284.48 109.22) (xy 287.02 109.22)
+		)
+		(stroke
+			(width 0)
+			(type default)
+		)
+	)
+	(wire
+		(pts
+			(xy 287.02 109.22) (xy 287.02 113.03)
+		)
+		(stroke
+			(width 0)
+			(type default)
+		)
+	)
+	(wire
+		(pts
 			(xy 147.32 196.85) (xy 147.32 203.2)
 		)
@@
 	(wire
 		(pts
+			(xy 294.64 109.22) (xy 294.64 113.03)
+		)
+		(stroke
+			(width 0)
+			(type default)
+		)
+	)
+	(wire
+		(pts
 			(xy 308.61 95.25) (xy 317.5 95.25)
 		)
@@
 	(wire
 		(pts
+			(xy 284.48 109.22) (xy 284.48 113.03)
+		)
+		(stroke
+			(width 0)
+			(type default)
+		)
+	)
+	(wire
+		(pts
 			(xy 299.72 87.63) (xy 308.61 87.63)
 		)
@@
 	(wire
 		(pts
+			(xy 289.56 109.22) (xy 289.56 113.03)
+		)
+		(stroke
+			(width 0)
+			(type default)
+		)
+	)
+	(wire
+		(pts
 			(xy 275.59 85.09) (xy 281.94 85.09)
 		)
@@
 	(wire
 		(pts
+			(xy 281.94 109.22) (xy 284.48 109.22)
+		)
+		(stroke
+			(width 0)
+			(type default)
+		)
+	)
+	(wire
+		(pts
 			(xy 299.72 95.25) (xy 308.61 95.25)
 		)
@@
 	(wire
 		(pts
+			(xy 292.1 109.22) (xy 292.1 113.03)
+		)
+		(stroke
+			(width 0)
+			(type default)
+		)
+	)
+	(wire
+		(pts
 			(xy 134.62 186.69) (xy 148.59 186.69)
 		)
@@
 		(pts
 			(xy 289.56 257.81) (xy 289.56 261.62)
+		)
+		(stroke
+			(width 0)
+			(type default)
+		)
+	)
+	(wire
+		(pts
+			(xy 287.02 109.22) (xy 289.56 109.22)
 		)
 		(stroke
@@
 					(unit 1)
 				)
+			)
+		)
+	)
+	(symbol
+		(lib_id "power:+3V3")
+		(at 289.56 105.41 270)
+		(unit 1)
+		(body_style 1)
+		(exclude_from_sim no)
+		(in_bom yes)
+		(on_board yes)
+		(in_pos_files yes)
+		(dnp no)
+		(fields_autoplaced yes)
+		(property "Reference" "#PWR012"
+			(at 285.75 105.41 0)
+			(hide yes)
+			(show_name no)
+			(do_not_autoplace no)
+			(effects
+				(font
+					(size 1.27 1.27)
+				)
+			)
+		)
+		(property "Value" "+3V3"
+			(at 293.37 105.4099 90)
+			(show_name no)
+			(do_not_autoplace no)
+			(effects
+				(font
+					(size 1.27 1.27)
+				)
+				(justify left)
+			)
+		)
+		(property "Footprint" ""
+			(at 289.56 105.41 0)
+			(hide yes)
+			(show_name no)
+			(do_not_autoplace no)
+			(effects
+				(font
+					(size 1.27 1.27)
+				)
+			)
+		)
+		(property "Datasheet" ""
+			(at 289.56 105.41 0)
+			(hide yes)
+			(show_name no)
+			(do_not_autoplace no)
+			(effects
+				(font
+					(size 1.27 1.27)
+				)
+			)
+		)
+		(property "Description" "Power symbol creates a global label with name \"+3V3\""
+			(at 289.56 105.41 0)
+			(hide yes)
+			(show_name no)
+			(do_not_autoplace no)
+			(effects
+				(font
+					(size 1.27 1.27)
+				)
+			)
+		)
+		(pin "1"
+		)
+		(instances
+			(project "SATVIK-26"
+				(path "/6d528f37-bbec-45e4-b49f-1b9f45291d26"
+					(reference "#PWR012")
+					(unit 1)
+				)

Commit message: Cezual update
Parts:
- added C16, C23, C24: 100nF, symbol Device:C
- added C17, C18: 47uF, symbol Device:C
- added C19: 3.3nF, symbol Device:C
- added C20: 100pF, symbol Device:C
- added C21, C22: 1uF, symbol Device:C
- added D1: B560/SS56, symbol Device:D_Schottky
- added D2: SMBJ26A, symbol Device:D_TVS
- added L1: 15uH, symbol Device:L
- added R4: 100k, symbol Device:R
- added R5: 52.3k, symbol Device:R
- added R6, R8: 10k, symbol Device:R
- added R7: 4.99k, symbol Device:R
- added R9: 1k, symbol Device:R
- added U3: AP2112K-3.3, Package_TO_SOT_SMD:SOT-23-5, symbol Regulator_Linear:AP2112K-3.3
Connections:
- net +3V3: now also C22.1, U3.5 (VOUT)
- net GND: now also U2.7 (GND), U2.9 (GND), C17.2, C18.2, C19.2, C20.2, C21.1, C22.2, C23.2, C24.1, D1.2 (A), D2.2 (A2), R4.2, R6.1, R9.2, U3.2 (GND)
- net VBAT_RAW: now reaches C6.2, C7.2, C9.2, R2.1, U2.2 (VIN)
- net VBAT_RAW: now also D2.1 (A1), R8.2
- net at U2.1 (BOOT): now also C16.1
- net at U2.4 (RT/CLK): now also R4.1
- net at U2.5 (FB): now also R5.2, R6.2
- net at U2.6 (COMP): now also C20.1, R7.1
- net at U2.8 (SW): now also C16.2, D1.1 (K), L1.1
- net at U1.15 (PC0): now also C23.1, R8.1, R9.1
- net CURR: now reaches U1.16 (PC1)
- net CURR: now also C24.2
- new net: C19.1, R7.2
- new net +5V: C17.1, C18.1, C21.2, L1.2, R5.1, U3.1 (VIN), U3.3 (EN)
Other:
- moved on the sheet: C10, C11, C12, C13, C14, C15, C6, C7, C8, C9, R2, R3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
