File: hardware/SATVIK-26/_autosave-SATVIK-26.kicad_pcb (KiCad board)
At the start: 4 copper layers, 36 x 36 mm, 78 parts, among them J1 Micro_SD_Card_Det1, J2 Conn_01x08_Pin, J3 Conn_01x06_Pin, J4 Conn_01x03_Pin, J5 Conn_01x04_Pin, J6 Conn_01x04_Pin, J7 Conn_01x04_Pin, SW1 SW_Push, SW2 SW_Push, U1 STM32H743VITx, U2 TPS54560BDDA, U3 AP2112K-3.3, U5 BMP388, U6 USBLC6-2SC6

Commit message: bruh
tis shi is hard :)
Parts:
- added U4: ICM-42688-P, easyeda2kicad:LGA-14_L3.0-W2.5-P0.50-TL, F.Cu at (80.2, 79.2)
- added Y1: Crystal, easyeda2kicad:CRYSTAL-SMD_4P-L3.2-W2.5-BL, F.Cu at (66.4, 74.6)
