File: hardware/SATVIK-26/SATVIK-26.kicad_pcb (KiCad board)
At the start: 4 copper layers, 36 x 36 mm, 78 parts, among them J1 Micro_SD_Card_Det1, J2 Conn_01x08_Pin, J3 Conn_01x06_Pin, J4 Conn_01x03_Pin, J5 Conn_01x04_Pin, J6 Conn_01x04_Pin, J7 Conn_01x04_Pin, SW1 SW_Push, SW2 SW_Push, U1 STM32H743VITx, U2 TPS54560BDDA, U3 AP2112K-3.3, U5 BMP388, U6 USBLC6-2SC6

Commit message: finnaly
Parts:
- added U4: ICM-42688-P, easyeda2kicad:LGA-14_L3.0-W2.5-P0.50-TL, F.Cu at (72.2, 74.3)
- added Y1: Crystal, easyeda2kicad:CRYSTAL-SMD_4P-L3.2-W2.5-BL, F.Cu at (65.3, 72.8)
- C14, C15, C16, C19, C20, C21, C30, R2, R3, R4, R5, R6, R7: moved to B.Cu
- moved R4 39.4 mm to (63.5, 49.8), turned to 180 degrees
- moved R5 34.7 mm to (73.0, 49.5), turned to 180 degrees
- moved R2 34.0 mm to (63.5, 51.8), turned to 180 degrees
- moved J4 31.0 mm to (82.0, 81.3), turned to 180 degrees
- moved R7 29.9 mm to (73.0, 51.5)
- moved R16 28.5 mm to (83.0, 55.3), turned to -90 degrees
- moved R8 27.9 mm to (63.0, 64.0)
- moved R1 27.6 mm to (78.8, 52.2)
- moved C20 27.5 mm to (73.0, 52.5), turned to 180 degrees
- moved C19 27.1 mm to (73.0, 53.5), turned to 180 degrees
- moved C10 27.0 mm to (83.0, 56.8), turned to 0 degrees
- moved C7 26.6 mm to (59.0, 57.5), turned to 180 degrees
- moved R3 26.3 mm to (63.5, 50.8), turned to 180 degrees
- moved D2 25.5 mm to (66.1, 61.5), turned to 0 degrees
- moved C2 25.5 mm to (84.0, 58.3)
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Routing:
- net GND: track 0.00 -> 130.1 mm, vias 1 -> 24
- net +5V: track 0.00 -> 109.4 mm, vias 0 -> 5
- net +3V3: track 0.00 -> 54.8 mm, vias 0 -> 10
- net /VBAT_RAW: track 0.00 -> 49.5 mm, vias 0 -> 2
- net /USART2_RX: track 0.00 -> 38.2 mm, vias 0 -> 2
- net /USART7_RX: track 0.00 -> 36.5 mm, vias 0 -> 2
- net /SD_D3: track 0.00 -> 34.9 mm, vias 0 -> 1
- net /USART2_TX: track 0.00 -> 33.8 mm, vias 0 -> 2
- net /USB_DM_MCU: track 0.00 -> 31.0 mm
- net /IMU_CS: track 0.00 -> 30.6 mm, vias 0 -> 2
- net /I2C2_SCL: track 0.00 -> 29.8 mm, vias 0 -> 2
- net /I2C2_SDA: track 0.00 -> 29.8 mm, vias 0 -> 3
- net /USB_DP_MCU: track 0.00 -> 29.3 mm
- net /UART4_RX: track 0.00 -> 29.2 mm, vias 0 -> 1
- net /USART6_RX: track 0.00 -> 28.0 mm, vias 0 -> 2
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
Commit message: Grant
Parts:
- moved C2 16.6 mm to (83.2, 41.7)
- moved R10 16.6 mm to (73.9, 58.7)
- moved R11 16.6 mm to (74.9, 58.7)
- moved R22 16.6 mm to (84.4, 63.7)
- moved U2 16.6 mm to (67.5, 35.0)
- moved U4 16.6 mm to (71.4, 57.7)
- moved C1 16.6 mm to (79.5, 56.5)
- moved C10 16.6 mm to (82.2, 40.2)
- moved C11 16.6 mm to (81.9, 55.5)
- moved C12 16.6 mm to (68.4, 57.0)
- moved C13 16.6 mm to (64.2, 51.2)
- moved C14 16.6 mm to (64.2, 51.2)
- moved C15 16.6 mm to (64.2, 49.7)
- moved C16 16.6 mm to (68.0, 38.2)
- moved C17 16.6 mm to (71.4, 41.7)
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Routing:
- net +3V3: track 54.8 -> 63.1 mm, vias 10 -> 11
- net GND: track 130.1 -> 134.9 mm, vias 24 -> 25
- net /IMU_CS: track 30.6 -> 26.5 mm
- net /SD_D3: track 34.9 -> 32.9 mm
- net /VBAT_RAW: track 49.5 -> 48.7 mm
- added copper zone on B.Cu, net GND
- added copper zone on F.Cu, net GND
Other:
- outline, holes or cut-outs redrawn
